File: hardware/LED.kicad_sch (KiCad schematic)
At the start: 64 parts, among them Q1 BSS138, Q2 BSS138

Commit message: HW: update to latest version
Parts:
- removed Q2: BSS138, Package_TO_SOT_SMD:SOT-23, symbol Transistor_FET:BSS138
- removed R119, R120: 10k, Resistor_SMD:R_0603_1608Metric, symbol Device:R_Small
- Q1: LCSC MFR (none) -> onsemi; LCSC MFR # (none) -> BSS138; LCSC Part # (none) -> C52895
Connections:
- net LED_OUT_DATA_5V: now also D24.1 (DOUT)
- net LED_IN_DATA renamed LED_DATA
- no-connect marks 2 -> 1
Other:
- company: (none) -> Avalution Engineering / Pollex
- title: (none) -> Zoutwachter Measurement-Switch
- moved on the sheet: C100, C101, C102, C103, C104, C105, C106, C108, C82, C84, C86, C88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
