File: hardware/Switch_ADG.kicad_sch (KiCad schematic)
At the start: 7 parts, among them U6 ADG6412BCPZ

Commit message: commit pending hw changes (rather old by now...)
Parts:
- renumbered C21 to C55, C22 to C56, R21 to R81, R22 to R82, R23 to R83, R24 to R84, U6 to U24

Commit message: HW: update to latest version
Parts:
- U9: renamed from U24; symbol ADG6412BCPZ:ADG6412BCPZ -> custom_library:ADG6412BCPZ; LCSC MFR - -> Analog Devices; LCSC MFR # - -> ADG6412BCPZ-REEL7; LCSC Part # - -> C5555803
- renumbered C55 to C27, C56 to C28, R81 to R21, R82 to R22, R83 to R23, R84 to R24
Other:
- company: (none) -> Avalution Engineering / Pollex
- title: (none) -> Zoutwachter Measurement-Switch
- moved on the sheet: C27, R21, R22, R23, R24, U9A
