File: hardware/USB.kicad_sch (KiCad schematic)
At the start: 12 parts, among them J6 USB-C Connector, U35 USBLC6-2SC6

Commit message: feat(RGB): WS2812B driver
Parts:
- C71, C73: footprint Capacitor_SMD:C_1210_3225Metric -> Capacitor_SMD:C_0603_1608Metric
- gave numbers to parts that had none: 1
Changed lines of the file:
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@@
       (effects (font (size 1.27 1.27)) (justify left))
     )
-    (property "Footprint" "Capacitor_SMD:C_1210_3225Metric" (at 217.17 37.465 0)
+    (property "Footprint" "Capacitor_SMD:C_0603_1608Metric" (at 217.17 37.465 0)
       (effects (font (size 1.27 1.27)) hide)
     )
@@
   (symbol (lib_id "Interface_USB:CP2102N-Axx-xQFN28") (at 235.585 74.93 0) (unit 1)
     (in_bom yes) (on_board yes) (dnp no) (fields_autoplaced)
-    (property "Reference" "U?" (at 237.7791 107.1301 0)
+    (property "Reference" "U36" (at 237.7791 107.1301 0)
       (effects (font (size 1.27 1.27)) (justify left))
     )
@@
     (instances
       (project "Zoutwachter-switch"
-        (path "/51927748-cbf3-4f36-990c-40014f3393ae"
-          (reference "U?") (unit 1)
-        )
         (path "/51927748-cbf3-4f36-990c-40014f3393ae/05dad072-cd43-486c-b27f-b8e24eeef930"
           (reference "U36") (unit 1)
@@
       (effects (font (size 1.27 1.27)) (justify left))
     )
-    (property "Footprint" "Capacitor_SMD:C_1210_3225Metric" (at 252.095 36.83 0)
-      (effects (font (size 1.27 1.27)) hide)
-    )
+    (property "Footprint" "Capacitor_SMD:C_0603_1608Metric" (at 252.095 36.83 0)
+      (effects (font (size 1.27 1.27)) hide)
+    )

Commit message: HW: update to latest version
Parts:
- J6: symbol Connector:USB_C_Receptacle_USB2.0 -> Connector:USB_C_Receptacle_USB2.0_16P
- renumbered U36 to U33, U35 to U34
Connections:
- net CTS renamed UART_USB_CTS
- net RTS renamed UART_USB_RTS
- net RX renamed UART_USB_RX
- net TX renamed UART_USB_TX
Other:
- company: (none) -> Avalution Engineering / Pollex
- title: (none) -> Zoutwachter Measurement-Switch
- moved on the sheet: C70, C71, C72, C73, J6, R14, R15, R16, R17, R18, U33
